Commit message: localize: enable recovery_manager_node (use_recovery default true)
localize.launch.py passed use_recovery:=false to bringup, so the
physical-stuck escape node never ran under the nav-chain launch the
runbook tells us to use. Near-wall room goals (e.g. domatio tou max)
then drive the footprint into ~99-cost inflation; the planner can no
longer plan (start-in-collision) and Nav2 loops raw Spin/BackUp until
ABORT.

HW-confirmed 2026-07-07 (kela3): with recovery_manager running it
detects the stuck (5s, ~0m displacement), does a BackUp to escape the
inflation pocket, and the re-issued goto to domatio tou max SUCCEEDS
with 0 recoveries. Spin-fix #1 (ax_max 2.0) also re-confirmed PASS in
the same session.

Adds a use_recovery launch arg (default true) and passes it through.

Co-Authored-By: Claude Opus 4.8 <noreply@anthropic.com>

File: description/robot_sim.urdf.xacro (robot description, xacro)
@@ -20,9 +20,9 @@
     </inertial>
     <collision>
-      <origin xyz="0 0 ${wheel_radius}"/>
+      <origin xyz="0 0 ${wheel_radius + body_height/2}"/>
       <geometry><cylinder radius="${body_radius}" length="${body_height}"/></geometry>
     </collision>
     <visual>
-      <origin xyz="0 0 ${wheel_radius}"/>
+      <origin xyz="0 0 ${wheel_radius + body_height/2}"/>
       <geometry><cylinder radius="${body_radius}" length="${body_height}"/></geometry>
       <material name="grey"><color rgba="0.2 0.2 0.22 1"/></material>

Commit message: sim: add a D435 stand-in (rgbd_camera) to the nav sim
No camera existed in the sim before (lidar + diff-drive only), so
rtabmap.launch.py could never be exercised against it — every 3D
mapping question had to wait for the real robot. camera_link matches
the real robot's measured mount (bringup.launch.py tf_base_camera:
x=0.14 z=0.586 pitch=0.525rad); a separate camera_color_optical_frame
child carries the pure REP103 rotation so RTAB-Map/image_geometry get
the frame convention they assume, without rotating the actual render
(gz's camera sensor looks along its own +X, confirmed against gz-sim8's
depth_camera_sensor.sdf example — nesting the sensor under the rotated
child would have pointed the render sideways). optical_frame_id on the
<camera> element relabels the message headers to that frame instead.

sim.launch.py bridges the rgbd_camera's image/depth_image/camera_info
and remaps them straight to the topic names rtabmap.launch.py already
expects (aligned_depth_to_color etc), so `ros2 launch home_robot
rtabmap.launch.py` works unmodified against the sim.

Used this to verify the anchor_frame=map fix (47de787) end-to-end with
real depth data on domain 77: after driving+turning, map->odom had
drifted ~1.9m/97deg (AMCL correction) while map->rtabmap_map stayed
pinned at identity throughout, and /rtabmap/cloud_map carried real
height (Z 0-0.56m, 7566 points) instead of the old flat Z=0. 424x240@15Hz
to keep this affordable on the machine's software (llvmpipe) rendering.

Co-Authored-By: Claude Sonnet 5 <noreply@anthropic.com>

File: description/robot_sim.urdf.xacro (robot description, xacro)
@@ -73,4 +73,25 @@
     <origin xyz="0 0 ${lidar_z}"/>
   </joint>
+  <!-- D435 stand-in, matching the real robot's measured mount
+       (bringup.launch.py tf_base_camera: x=0.14 z=0.586 pitch=0.525 rad
+       / 30.1deg down — see [[project_robot_camera_pitch_wrong]]).
+       camera_link keeps the normal X-forward/Z-up body convention (what the
+       gz sensor plugin actually renders along); camera_color_optical_frame
+       is a pure REP103 rotation (Z-forward/X-right/Y-down, no extra
+       translation) so RTAB-Map/image_geometry get the frame they assume —
+       the sensor itself attaches to camera_link with optical_frame_id
+       pointed at the rotated frame below, not by moving the render pose. -->
+  <link name="camera_link"/>
+  <joint name="camera_joint" type="fixed">
+    <parent link="base_link"/>
+    <child link="camera_link"/>
+    <origin xyz="0.14 0 0.586" rpy="0 0.525 0"/>
+  </joint>
+  <link name="camera_color_optical_frame"/>
+  <joint name="camera_optical_joint" type="fixed">
+    <parent link="camera_link"/>
+    <child link="camera_color_optical_frame"/>
+    <origin xyz="0 0 0" rpy="-1.5707963 0 -1.5707963"/>
+  </joint>
   <!-- ── Gazebo: diff-drive + lidar sensor ───────────────────────── -->
   <gazebo>
@@ -109,3 +130,32 @@
     </sensor>
   </gazebo>
+  <!-- D435 stand-in: rgbd_camera sensor attached to the PHYSICAL link
+       (camera_link, X-forward — this is the axis gz actually renders
+       along; confirmed against gz-sim8's own depth_camera_sensor.sdf
+       example, where a pure yaw rotation alone re-aimed the view, which
+       only makes sense if the render axis is local +X, not OpenGL -Z).
+       optical_frame_id only relabels the message headers to the REP103
+       frame defined above in the URDF — it does not move the render, so
+       this keeps the true 30.1deg-down tilt while still handing RTAB-Map
+       a properly-oriented optical frame. Modest 424x240 res + 15Hz: this
+       machine renders in software (llvmpipe, no GPU) and RGBD is much
+       heavier per-frame than the lidar. -->
+  <gazebo reference="camera_link">
+    <sensor name="camera" type="rgbd_camera">
+      <update_rate>15</update_rate>
+      <topic>camera</topic>
+      <camera>
+        <horizontal_fov>1.2043</horizontal_fov>
+        <image>
+          <width>424</width>
+          <height>240</height>
+          <format>R8G8B8</format>
+        </image>
+        <clip><near>0.1</near><far>8.0</far></clip>
+        <optical_frame_id>camera_color_optical_frame</optical_frame_id>
+      </camera>
+      <always_on>1</always_on>
+      <visualize>true</visualize>
+    </sensor>
+  </gazebo>
 </robot>
